File: LED-mini20-SHIM.brd (EAGLE design)
At the start: 50.8 x 12.7 mm, 26 parts, among them IC1 TXB0101DCKR

Commit message: Updated texts. Generated CAM files. Generated PNG preview. Generated PDF schematics.
Other:
- board text added: "LED-mini20-SHIM v.1.0"
- board text removed: "LED-mini-SHIM v.1.0"
Changed lines of the file:
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@@
 <wire x1="0" y1="11.43" x2="1.27" y2="12.7" width="0" layer="20" curve="-90"/>
 <wire x1="49.53" y1="12.7" x2="50.8" y2="11.43" width="0" layer="20" curve="-90"/>
-<text x="16.129" y="6.731" size="1.27" layer="21" font="vector" ratio="24">LED-mini-SHIM v.1.0</text>
+<text x="16.129" y="6.731" size="1.27" layer="21" font="vector" ratio="24">LED-mini20-SHIM v.1.0</text>
 <rectangle x1="0" y1="0" x2="2.54" y2="2.54" layer="21" rot="R90"/>
 <text x="2.794" y="4.445" size="0.6096" layer="21" font="vector" ratio="12" rot="R90">2</text>
