File: LED-plus20-SHIM.brd (EAGLE design)
At the start: 56 x 65 mm, 306 parts, among them IC1 TXB0101DCKR

Commit message: Updated texts. Generated CAM files. Generated PNG preview. Generated PDF schematics.
Other:
- board text added: "LED-plus20-SHIM v1.0"
- board text removed: "LED-plus-SHIM v1.0"
Changed lines of the file:
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@@
 <drawing>
 <settings>
-<setting alwaysvectorfont="yes"/>
+<setting alwaysvectorfont="no"/>
 <setting verticaltext="up"/>
 </settings>
@@
 <wire x1="0" y1="2.9972" x2="0" y2="3" width="0" layer="20" curve="-0.053476"/>
 <wire x1="0" y1="62" x2="0" y2="62.0014" width="0" layer="20" curve="-0.026738"/>
-<text x="37.92" y="3.398" size="1.27" layer="21" font="vector" ratio="24" rot="R180">LED-plus-SHIM v1.0</text>
+<text x="38.1" y="3.429" size="1.27" layer="21" font="vector" ratio="24" rot="R180">LED-plus20-SHIM v1.0</text>
 <text x="34.724" y="46.513" size="1.016" layer="22" font="vector" ratio="12" rot="MR0">http://redscorp.net</text>
 <text x="34.724" y="45.243" size="1.016" layer="22" font="vector" ratio="12" rot="MR0">(c) Andriy Golovnya</text>
