File: LED-plus20-SHIM.sch (EAGLE design)
At the start: 305 parts, among them IC1 TXB0101DCKR

Commit message: Updated texts. Generated CAM files. Generated PNG preview. Generated PDF schematics.
Other:
- note added: "PI-LEDP20S-0010"
- note removed: "PI-LEDPS-0010"
Changed lines of the file:
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@@
 <plain>
 <text x="256.54" y="7.62" size="2.54" layer="94">1.0</text>
-<text x="198.12" y="7.62" size="2.54" layer="94">PI-LEDPS-0010</text>
+<text x="198.12" y="7.62" size="2.54" layer="94">PI-LEDP20S-0010</text>
 <text x="165.1" y="25.4" size="2.54" layer="94">Pi Plus sized LED-SHIM for Pi's 40-pin extension slot
 (c) Andriy Golovnya</text>
@@
 <plain>
 <text x="256.54" y="7.62" size="2.54" layer="94">1.0</text>
-<text x="198.12" y="7.62" size="2.54" layer="94">PI-LEDPS-0010</text>
+<text x="198.12" y="7.62" size="2.54" layer="94">PI-LEDP20S-0010</text>
 <text x="165.1" y="25.4" size="2.54" layer="94">Pi Plus sized LED-SHIM for Pi's 40-pin extension slot
 (c) Andriy Golovnya</text>
@@
 <plain>
 <text x="256.54" y="7.62" size="2.54" layer="94">1.0</text>
-<text x="198.12" y="7.62" size="2.54" layer="94">PI-LEDPS-0010</text>
+<text x="198.12" y="7.62" size="2.54" layer="94">PI-LEDP20S-0010</text>
 <text x="165.1" y="25.4" size="2.54" layer="94">Pi Plus sized LED-SHIM for Pi's 40-pin extension slot
 (c) Andriy Golovnya</text>
@@
 <plain>
 <text x="256.54" y="7.62" size="2.54" layer="94">1.0</text>
-<text x="198.12" y="7.62" size="2.54" layer="94">PI-LEDPS-0010</text>
+<text x="198.12" y="7.62" size="2.54" layer="94">PI-LEDP20S-0010</text>
 <text x="165.1" y="25.4" size="2.54" layer="94">Pi Plus sized LED-SHIM for Pi's 40-pin extension slot
 (c) Andriy Golovnya</text>
