File: LED-zero20-SHIM.brd (EAGLE design)
At the start: 30 x 65 mm, 157 parts, among them IC1 TXB0101DCKR

Commit message: Updated texts. Generated CAM files. Generated PNG preview. Generated PDF schematics.
Other:
- board text added: "LED-zero20-SHIM v1.0"
- board text removed: "LED-zero-SHIM v1.0"
Changed lines of the file:
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@@
 <drawing>
 <settings>
-<setting alwaysvectorfont="no"/>
+<setting alwaysvectorfont="yes"/>
 <setting verticaltext="up"/>
 </settings>
@@
 <circle x="26.5" y="61.5" radius="3.2" width="0" layer="29"/>
 <circle x="26.5" y="61.5" radius="3.2" width="0" layer="30"/>
-<text x="21.537" y="42.83" size="1.27" layer="22" font="vector" ratio="24" rot="MR0">LED-zero-SHIM v1.0</text>
+<text x="22.352" y="42.799" size="1.27" layer="22" font="vector" ratio="24" rot="MR0">LED-zero20-SHIM v1.0</text>
 <text x="19.357" y="49.307" size="1.016" layer="22" font="vector" ratio="12" rot="MR0">http://redscorp.net</text>
 <text x="19.357" y="48.037" size="1.016" layer="22" font="vector" ratio="12" rot="MR0">(c) Andriy Golovnya</text>
